Commit message: affichage rviz ok

File: urdf/zumo.urdf (robot description, URDF)
Before this commit: robot Zumo de Compet, 1 links, 0 joints
Links:
- added link base; visual mesh filename=package://Zumo2Compet/urdf/zumo.STL scale=1 1 1
- link base_link: geometry 
Joints:
- added joint joint1: type fixed, parent base_link, child base

Commit message: affichage rviz

File: urdf/zumo.urdf (robot description, URDF)
Before this commit: robot Zumo de Compet, 2 links, 1 joints
Joints:
- joint joint1: axis (none) -> 0 0 1; origin (none) -> xyz=0 0 0 rpy=0 0 0; type fixed -> planar
